File: Schematy/diagrams/light/light.kicad_sch (KiCad schematic)
At the start: 5 parts

Commit message: Basic setup
Parts:
- gave numbers to parts that had none: 1
Changed lines of the file:
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@@
   (symbol (lib_id "Transistor_FET:2N7000") (at 54.61 43.18 0) (unit 1)
     (in_bom yes) (on_board yes) (fields_autoplaced)
-    (property "Reference" "Q?" (id 0) (at 60.96 41.9099 0)
+    (property "Reference" "Q1" (id 0) (at 60.96 41.9099 0)
       (effects (font (size 1.27 1.27)) (justify left))
     )
@@
     )
     (path "/29329e0a-8809-4ca4-b945-9734a0c3cf89"
-      (reference "Q?") (unit 1) (value "2N7000") (footprint "Package_TO_SOT_THT:TO-92_Inline")
+      (reference "Q1") (unit 1) (value "2N7000") (footprint "Package_TO_SOT_THT:TO-92_Inline")
     )
     (path "/c0a86600-d199-4e8a-9a12-c864156662da"
